Commit message: First attempt at pan/tilt in the robot model
Currently you can see it panning in rviz but the tilt doesn't work. And,
the position and size of the pan/tilt servos are probably wrong.

File: robots/kobuki_hexagons_astra.urdf.xacro (robot description, xacro)
@@ -10,6 +10,8 @@
   <xacro:include filename="$(find ras_description)/urdf/stacks/hexagons.urdf.xacro"/>
   <xacro:include filename="$(find ras_description)/urdf/sensors/astra.urdf.xacro"/>
+  <xacro:include filename="$(find ras_description)/urdf/pantilt.urdf.xacro"/>
   <kobuki/>
   <stack_hexagons parent="base_link"/>
-  <sensor_astra parent="base_link"/>
+  <pantilt parent="base_link"/>
+  <sensor_astra parent="pantilt_camera_link"/>
 </robot>

File: urdf/turtlebot_properties.urdf.xacro (robot description, xacro)
@@ -20,8 +20,8 @@
    -->
 	<!--<xacro:property name="cam_px" value="-0.087" />-->
-	<xacro:property name="cam_px" value="0.0635" />
+	<xacro:property name="cam_px" value="0" />
 <!--	<xacro:property name="cam_py" value="-0.0125" /> Y varies for different configurations. get sets in sensors_urdf -->
 	<!--<xacro:property name="cam_pz" value="0.2870" />-->
-	<xacro:property name="cam_pz" value="1.4224" />
+	<xacro:property name="cam_pz" value="0" />
 	<xacro:property name="cam_or" value="0" />
 	<xacro:property name="cam_op" value="0" />

Commit message: Fairly accurate now
When running demo_pan_tilt.py, the objects stay in almost the same place when
viewing the PointCloud2 in rviz.

File: robots/kobuki_hexagons_astra.urdf.xacro (robot description, xacro)
@@ -14,4 +14,4 @@
   <stack_hexagons parent="base_link"/>
   <pantilt parent="base_link"/>
-  <sensor_astra parent="pantilt_camera_link"/>
+  <sensor_astra parent="tilt_link"/>
 </robot>

File: urdf/pantilt.urdf.xacro (robot description, xacro)
@@ -1,81 +1,82 @@
 <?xml version="1.0"?>
 <robot name="pantilt" xmlns:xacro="http://ros.org/wiki/xacro">
-  <xacro:macro name="pantilt" params="parent">
-	<!-- camera -->
-	<!-- Based on: https://answers.ros.org/question/142366/simulating-a-camera-with-a-pan-tilt-unit/ -->
-	<!-- i think the pan joint can be deleted-->
-<!-- TODO name these what ArbotiX-M controller named them, so we have their values... -->
-	<!-- pan? -->
-	<joint name="head_pan_joint" type="fixed">
-	    <axis xyz="0 1 0" />
-	    <origin xyz="0.0635 0 1.4224" rpy="0 0 0"/> <!-- you have to measure these relative to parent, given in meters -->
-	    <parent link="${parent}"/>
-	    <child link="pan_link"/>
-	  </joint>
-	<!-- tilt? -->
-	<joint name="head_tilt_joint" type="revolute">
-	    <axis xyz="0 0 1" />
-	  <limit lower="-${M_PI/2}" upper="${M_PI/2}"  effort="50" velocity="1"/>
-	    <origin xyz="0.0 0 0.08" rpy="0 0 0"/>
-	    <parent link="pan_link"/>
-	    <child link="pantilt_camera_link"/>
-	  </joint>
-	<link name="pan_link">
-	    <collision>
-	      <origin xyz="0 0 0" rpy="0 0 0"/>
-	      <geometry>
-	    <box size="0.16 0.16 0.01"/>
-	      </geometry>
-	    </collision>
-	    <visual>
-	      <origin xyz="0 0 0" rpy="0 0 0"/>
-	      <geometry>
-		    <box size="0.02 0.02 0.01"/> <!-- 0.16 0.16 0.01 -->
-	      </geometry>
-	    </visual>
-	    <inertial>
-	      <mass value="1e-5" />
-	      <origin xyz="0 0 0" rpy="0 0 0"/>
-	      <inertia ixx="1e-6" ixy="0" ixz="0" iyy="1e-6" iyz="0" izz="1e-6" />
-	    </inertial>
-	  </link>
-	    <gazebo reference="pan_link">
-		<material>Gazebo/Yellow</material>
-	    </gazebo>
-	<link name="pantilt_camera_link">
-	    <collision>
-	      <origin xyz="0 0 0" rpy="0 0 0"/>
-	      <geometry>
-	    <box size="0.05 0.05 0.05"/>
-	      </geometry>
-	    </collision>
-	    <visual>
-	      <origin xyz="0 0 0" rpy="0 0 0"/>
-	      <geometry>
-	    <box size="0.05 0.05 0.05"/>
-	      </geometry>
-	    </visual>
-	    <inertial>
-	      <mass value="1e-5" />
-	      <origin xyz="0 0 0" rpy="0 0 0"/>
-	      <inertia ixx="1e-6" ixy="0" ixz="0" iyy="1e-6" iyz="0" izz="1e-6" />
-	    </inertial>
-	  </link>
-	    <gazebo reference="pantilt_camera_link">
-		<material>Gazebo/Red</material>
-	    </gazebo>
-	<transmission name="pan_trans">
-	  <type>transmission_interface/SimpleTransmission</type>
-	  <joint name="head_tilt_joint"/>
-	  <actuator name="camera_pan_unit">
-	    <hardwareInterface>EffortJointInterface</hardwareInterface>
-	    <mechanicalReduction>1</mechanicalReduction>
-	  </actuator>
-	</transmission>
-	<gazebo>
-	  <plugin name="gazebo_ros_control" filename="libgazebo_ros_control.so">
-	    <robotNamespace>/aircobot</robotNamespace><!--seems to work-->
-	  </plugin>
-	</gazebo>
-  </xacro:macro>
+    <xacro:macro name="pantilt" params="parent">
+        <!-- Based on: https://answers.ros.org/question/142366/simulating-a-camera-with-a-pan-tilt-unit/ -->
+        <joint name="head_pan_joint" type="revolute">
+            <axis xyz="0 0 1" />
+            <limit lower="-${M_PI/2}" upper="${M_PI/2}"  effort="50" velocity="1"/>
+            <!--
+                 Measure these relative to parent
+                 These are w.r.t. base_link (the parent), given in meters
+                 This is to center of the rotating part of the bottom (pan) servo.
+                 -->
+            <origin xyz="0.0381 0 1.3081" rpy="0 0 0"/>
+            <parent link="${parent}"/>
+            <child link="pan_link"/>
+        </joint>
+        <joint name="head_tilt_joint" type="revolute">
+            <axis xyz="0 1 0" />
+            <limit lower="-${M_PI/2}" upper="${M_PI/2}"  effort="50" velocity="1"/>
+            <origin xyz="0.0169 0 0.01905" rpy="0 -0.25 0"/>
+            <parent link="pan_link"/>
+            <child link="tilt_link"/>
+        </joint>
+        <link name="pan_link">
+            <collision>
+                <origin xyz="0 0 0" rpy="0 0 0"/>
+                <geometry>
+                    <box size="0.03175 0.0508 0.03175"/>
+                </geometry>
+            </collision>
+            <visual>
+                <origin xyz="0 0 0" rpy="0 0 0"/>
+                <geometry>
+                    <box size="0.03175 0.0508 0.03175"/>
+                </geometry>
+            </visual>
+            <inertial>
+                <mass value="1e-5" />
+                <origin xyz="0 0 0" rpy="0 0 0"/>
+                <inertia ixx="1e-6" ixy="0" ixz="0" iyy="1e-6" iyz="0" izz="1e-6" />
+            </inertial>
+        </link>
+        <gazebo reference="pan_link">
+            <material>Gazebo/Yellow</material>
+        </gazebo>
+        <link name="tilt_link">
+            <collision>
+                <origin xyz="0 0 0" rpy="0 0 0"/>
+                <geometry>
+                    <box size="0.0254 0.0508 0.0381"/>
+                </geometry>
+            </collision>
+            <visual>
+                <origin xyz="0 0 0" rpy="0 0 0"/>
+                <geometry>
+                    <box size="0.0254 0.0508 0.0381"/>
+                </geometry>
+            </visual>
+            <inertial>
+                <mass value="1e-5" />
+                <origin xyz="0 0 0" rpy="0 0 0"/>
+                <inertia ixx="1e-6" ixy="0" ixz="0" iyy="1e-6" iyz="0" izz="1e-6" />
+            </inertial>
+        </link>
+        <gazebo reference="tilt_link">
+            <material>Gazebo/Red</material>
+        </gazebo>
+        <transmission name="pan_trans">
+            <type>transmission_interface/SimpleTransmission</type>
+            <joint name="head_tilt_joint"/>
+            <actuator name="camera_pan_unit">
+                <hardwareInterface>EffortJointInterface</hardwareInterface>
+                <mechanicalReduction>1</mechanicalReduction>
+            </actuator>
+        </transmission>
+        <gazebo>
+            <plugin name="gazebo_ros_control" filename="libgazebo_ros_control.so">
+                <robotNamespace>/aircobot</robotNamespace><!--seems to work-->
+            </plugin>
+        </gazebo>
+    </xacro:macro>
 </robot>
